File: vco.kicad_sch (KiCad schematic)
At the start: 10 parts, among them J1 AudioPlug2, U1 40106, U2 TL074

Commit message: gi
Connections:
- net GND: now also J1.S, R4.1
- net at C2.2, R2.1: now also R3.1
- net at R4.2: now also J1.T, R3.2
Other:
- moved on the sheet: R3, R4
Changed lines of the file:
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@@
   (junction (at 154.94 113.03) (diameter 0) (color 0 0 0 0)
   )
+  (junction (at 184.785 113.03) (diameter 0) (color 0 0 0 0)
+  )
+  (wire (pts (xy 224.155 124.46) (xy 216.535 124.46))
+    (stroke (width 0) (type default))
+  )
   (wire (pts (xy 154.94 113.03) (xy 157.48 113.03))
     (stroke (width 0) (type default))
@@
     (stroke (width 0) (type default))
   )
-  (wire (pts (xy 168.275 113.03) (xy 187.325 113.03))
+  (wire (pts (xy 168.275 113.03) (xy 173.99 113.03))
     (stroke (width 0) (type default))
   )
@@
     (stroke (width 0) (type default))
   )
+  (wire (pts (xy 224.155 119.38) (xy 217.805 119.38))
+    (stroke (width 0) (type default))
+  )
+  (wire (pts (xy 216.535 124.46) (xy 216.535 130.175))
+    (stroke (width 0) (type default))
+  )
+  (wire (pts (xy 184.785 113.03) (xy 184.785 116.84))
+    (stroke (width 0) (type default))
+  )
   (wire (pts (xy 100.33 111.76) (xy 100.33 119.38))
     (stroke (width 0) (type default))
@@
     (stroke (width 0) (type default))
   )
+  (wire (pts (xy 217.805 119.38) (xy 217.805 113.03))
+    (stroke (width 0) (type default))
+  )
   (wire (pts (xy 168.275 113.03) (xy 168.275 116.205))
     (stroke (width 0) (type default))
@@
     (stroke (width 0) (type default))
   )
+  (wire (pts (xy 184.785 113.03) (xy 217.805 113.03))
+    (stroke (width 0) (type default))
+  )
   (wire (pts (xy 100.33 104.14) (xy 100.33 99.06))
     (stroke (width 0) (type default))
   )
   (wire (pts (xy 165.1 67.31) (xy 129.54 67.31))
+    (stroke (width 0) (type default))
+  )
+  (wire (pts (xy 181.61 113.03) (xy 184.785 113.03))
     (stroke (width 0) (type default))
   )
@@
     )
   )
+  (symbol (lib_id "power:GND") (at 216.535 130.175 0) (unit 1)
+    (in_bom yes) (on_board yes) (dnp no) (fields_autoplaced)
+    (property "Reference" "#PWR05" (at 216.535 136.525 0)
+      (effects (font (size 1.27 1.27)) hide)
+    )
+    (property "Value" "GND" (at 216.535 135.255 0)
+      (effects (font (size 1.27 1.27)))
+    )
+    (property "Footprint" "" (at 216.535 130.175 0)
+      (effects (font (size 1.27 1.27)) hide)
+    )
+    (property "Datasheet" "" (at 216.535 130.175 0)
+      (effects (font (size 1.27 1.27)) hide)
+    )
+    (pin "1")
+    (instances
+      (project "vco"
+        (path "/6034af30-8876-4e85-84ef-45b5f1065c0a"
+          (reference "#PWR05") (unit 1)
+        )
+      )
+    )
+  )
   (symbol (lib_id "Device:R") (at 168.275 120.015 0) (unit 1)
     (in_bom yes) (on_board yes) (dnp no) (fields_autoplaced)
@@
         (path "/6034af30-8876-4e85-84ef-45b5f1065c0a"
           (reference "R1") (unit 1)
+        )
+      )
+    )
+  )
+  (symbol (lib_id "power:GND") (at 184.785 124.46 0) (unit 1)
+    (in_bom yes) (on_board yes) (dnp no) (fields_autoplaced)
+    (property "Reference" "#PWR04" (at 184.785 130.81 0)
+      (effects (font (size 1.27 1.27)) hide)
+    )
+    (property "Value" "GND" (at 184.785 129.54 0)
+      (effects (font (size 1.27 1.27)))
+    )
+    (property "Footprint" "" (at 184.785 124.46 0)
+      (effects (font (size 1.27 1.27)) hide)
+    )
+    (property "Datasheet" "" (at 184.785 124.46 0)
+      (effects (font (size 1.27 1.27)) hide)
+    )
+    (pin "1")
+    (instances
+      (project "vco"
+        (path "/6034af30-8876-4e85-84ef-45b5f1065c0a"
+          (reference "#PWR04") (unit 1)
         )
       )
@@
     )
   )
-  (symbol (lib_id "Device:R") (at 101.6 139.7 0) (unit 1)
-    (in_bom yes) (on_board yes) (dnp no) (fields_autoplaced)
-    (property "Reference" "R4" (at 104.14 138.43 0)
-      (effects (font (size 1.27 1.27)) (justify left))
-    )
-    (property "Value" "R" (at 104.14 140.97 0)
-      (effects (font (size 1.27 1.27)) (justify left))
-    )
-    (property "Footprint" "" (at 99.822 139.7 90)
-      (effects (font (size 1.27 1.27)) hide)
-    )
-    (property "Datasheet" "~" (at 101.6 139.7 0)
+  (symbol (lib_id "Device:R") (at 184.785 120.65 180) (unit 1)
+    (in_bom yes) (on_board yes) (dnp no) (fields_autoplaced)
+    (property "Reference" "R4" (at 187.325 119.38 0)
+      (effects (font (size 1.27 1.27)) (justify right))
+    )
+    (property "Value" "R" (at 187.325 121.92 0)
+      (effects (font (size 1.27 1.27)) (justify right))
+    )
+    (property "Footprint" "" (at 186.563 120.65 90)
+      (effects (font (size 1.27 1.27)) hide)
+    )
+    (property "Datasheet" "~" (at 184.785 120.65 0)
       (effects (font (size 1.27 1.27)) hide)
     )
@@
     )
   )
-  (symbol (lib_id "Device:R") (at 85.09 137.16 0) (unit 1)
-    (in_bom yes) (on_board yes) (dnp no) (fields_autoplaced)
-    (property "Reference" "R3" (at 87.63 135.89 0)
-      (effects (font (size 1.27 1.27)) (justify left))
-    )
-    (property "Value" "R" (at 87.63 138.43 0)
-      (effects (font (size 1.27 1.27)) (justify left))
-    )
-    (property "Footprint" "" (at 83.312 137.16 90)
-      (effects (font (size 1.27 1.27)) hide)
-    )
-    (property "Datasheet" "~" (at 85.09 137.16 0)
-      (effects (font (size 1.27 1.27)) hide)
-    )
+  (symbol (lib_id "Device:R") (at 177.8 113.03 90) (unit 1)
+    (in_bom yes) (on_board yes) (dnp no) (fields_autoplaced)
+    (property "Reference" "R3" (at 177.8 107.315 90)
+      (effects (font (size 1.27 1.27)))
+    )
+    (property "Value" "R" (at 177.8 109.855 90)
+      (effects (font (size 1.27 1.27)))
+    )
+    (property "Footprint" "" (at 177.8 114.808 90)
+      (effects (font (size 1.27 1.27)) hide)
+    )
+    (property "Datasheet" "~" (at 177.8 113.03 0)
+      (effects (font (size 1.27 1.27)) hide)
+    )

Commit message: pot on npn
Parts:
- added Q1: BC548C, BC548C:TO92250P510H770-3, symbol BC548C:BC548C
- added R5, R6, R7, R8, R9: R, symbol Device:R
- added RV1: R_Potentiometer, symbol Device:R_Potentiometer
Changed lines of the file:
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@@
+    )
+  )
+  (symbol (lib_id "Device:R") (at 211.455 149.225 0) (unit 1)
+    (in_bom yes) (on_board yes) (dnp no) (fields_autoplaced)
+    (property "Reference" "R8" (at 213.995 147.955 0)
+      (effects (font (size 1.27 1.27)) (justify left))
+    )
+    (property "Value" "R" (at 213.995 150.495 0)
+      (effects (font (size 1.27 1.27)) (justify left))
+    )
+    (property "Footprint" "" (at 209.677 149.225 90)
+      (effects (font (size 1.27 1.27)) hide)
+    )
+    (property "Datasheet" "~" (at 211.455 149.225 0)
+      (effects (font (size 1.27 1.27)) hide)
+    )
+    (pin "1")
+    (pin "2")
+    (instances
+      (project "vco"
+        (path "/6034af30-8876-4e85-84ef-45b5f1065c0a"
+          (reference "R8") (unit 1)
+        )
+      )
     )
   )
@@
     )
   )
+  (symbol (lib_id "BC548C:BC548C") (at 201.93 74.93 0) (unit 1)
+    (in_bom yes) (on_board yes) (dnp no) (fields_autoplaced)
+    (property "Reference" "Q1" (at 205.74 73.66 0)
+      (effects (font (size 1.27 1.27)) (justify left))
+    )
+    (property "Value" "BC548C" (at 205.74 76.2 0)
+      (effects (font (size 1.27 1.27)) (justify left))
+    )
+    (property "Footprint" "BC548C:TO92250P510H770-3" (at 201.93 74.93 0)
+      (effects (font (size 1.27 1.27)) (justify bottom) hide)
+    )
+    (property "Datasheet" "" (at 201.93 74.93 0)
+      (effects (font (size 1.27 1.27)) hide)
+    )
+    (property "MF" "ON" (at 201.93 74.93 0)
+      (effects (font (size 1.27 1.27)) (justify bottom) hide)
+    )
+    (property "Purchase-URL" "https://www.snapeda.com/api/url_track_click_mouser/?unipart_id=455158&manufacturer=ON&part_name=BC548C&search_term=None" (at 201.93 74.93 0)
+      (effects (font (size 1.27 1.27)) (justify bottom) hide)
+    )
+    (property "Package" "E-PKG AXIAL-LEADED-2 ON Semiconductor" (at 201.93 74.93 0)
+      (effects (font (size 1.27 1.27)) (justify bottom) hide)
+    )
+    (property "Price" "None" (at 201.93 74.93 0)
+      (effects (font (size 1.27 1.27)) (justify bottom) hide)
+    )
+    (property "Check_prices" "https://www.snapeda.com/parts/BC548C/Onsemi/view-part/?ref=eda" (at 201.93 74.93 0)
+      (effects (font (size 1.27 1.27)) (justify bottom) hide)
+    )
+    (property "SnapEDA_Link" "https://www.snapeda.com/parts/BC548C/Onsemi/view-part/?ref=snap" (at 201.93 74.93 0)
+      (effects (font (size 1.27 1.27)) (justify bottom) hide)
+    )
+    (property "MP" "BC548C" (at 201.93 74.93 0)
+      (effects (font (size 1.27 1.27)) (justify bottom) hide)
+    )
+    (property "Availability" "In Stock" (at 201.93 74.93 0)
+      (effects (font (size 1.27 1.27)) (justify bottom) hide)
+    )
+    (property "Description" "\nBipolar (BJT) Transistor NPN 30 V 100 mA 300MHz 625 mW Through Hole TO-92 (TO-226)\n" (at 201.93 74.93 0)
+      (effects (font (size 1.27 1.27)) (justify bottom) hide)
+    )
+    (pin "1")
+    (pin "2")
+    (pin "3")
+    (instances
+      (project "vco"
+        (path "/6034af30-8876-4e85-84ef-45b5f1065c0a"
+          (reference "Q1") (unit 1)
+        )
+      )
+    )
+  )
+  (symbol (lib_id "Device:R") (at 182.88 150.495 0) (unit 1)
+    (in_bom yes) (on_board yes) (dnp no) (fields_autoplaced)
+    (property "Reference" "R6" (at 185.42 149.225 0)
+      (effects (font (size 1.27 1.27)) (justify left))
+    )
+    (property "Value" "R" (at 185.42 151.765 0)
+      (effects (font (size 1.27 1.27)) (justify left))
+    )
+    (property "Footprint" "" (at 181.102 150.495 90)
+      (effects (font (size 1.27 1.27)) hide)
+    )
+    (property "Datasheet" "~" (at 182.88 150.495 0)
+      (effects (font (size 1.27 1.27)) hide)
+    )
+    (pin "1")
+    (pin "2")
+    (instances
+      (project "vco"
+        (path "/6034af30-8876-4e85-84ef-45b5f1065c0a"
+          (reference "R6") (unit 1)
+        )
+      )
+    )
+  )
   (symbol (lib_id "Device:R") (at 184.785 120.65 180) (unit 1)
     (in_bom yes) (on_board yes) (dnp no) (fields_autoplaced)
@@
     )
   )
+  (symbol (lib_id "Device:R") (at 226.06 149.225 0) (unit 1)
+    (in_bom yes) (on_board yes) (dnp no) (fields_autoplaced)
+    (property "Reference" "R9" (at 228.6 147.955 0)
+      (effects (font (size 1.27 1.27)) (justify left))
+    )
+    (property "Value" "R" (at 228.6 150.495 0)
+      (effects (font (size 1.27 1.27)) (justify left))
+    )
+    (property "Footprint" "" (at 224.282 149.225 90)
+      (effects (font (size 1.27 1.27)) hide)
+    )
+    (property "Datasheet" "~" (at 226.06 149.225 0)
+      (effects (font (size 1.27 1.27)) hide)
+    )
+    (pin "1")
+    (pin "2")
+    (instances
+      (project "vco"
+        (path "/6034af30-8876-4e85-84ef-45b5f1065c0a"
+          (reference "R9") (unit 1)
+        )
+      )
+    )
+  )
+  (symbol (lib_id "Device:R") (at 196.85 148.59 0) (unit 1)
+    (in_bom yes) (on_board yes) (dnp no) (fields_autoplaced)
+    (property "Reference" "R7" (at 199.39 147.32 0)
+      (effects (font (size 1.27 1.27)) (justify left))
+    )
+    (property "Value" "R" (at 199.39 149.86 0)
+      (effects (font (size 1.27 1.27)) (justify left))
+    )
+    (property "Footprint" "" (at 195.072 148.59 90)
+      (effects (font (size 1.27 1.27)) hide)
+    )
+    (property "Datasheet" "~" (at 196.85 148.59 0)
+      (effects (font (size 1.27 1.27)) hide)
+    )
+    (pin "1")
+    (pin "2")
+    (instances
+      (project "vco"
+        (path "/6034af30-8876-4e85-84ef-45b5f1065c0a"
+          (reference "R7") (unit 1)
+        )
+      )
+    )
+  )
   (symbol (lib_id "Device:C") (at 114.3 107.95 0) (unit 1)
     (in_bom yes) (on_board yes) (dnp no) (fields_autoplaced)
@@
     )
   )
+  (symbol (lib_id "Device:R") (at 168.91 150.495 0) (unit 1)
+    (in_bom yes) (on_board yes) (dnp no) (fields_autoplaced)
+    (property "Reference" "R5" (at 171.45 149.225 0)
+      (effects (font (size 1.27 1.27)) (justify left))
+    )
+    (property "Value" "R" (at 171.45 151.765 0)
+      (effects (font (size 1.27 1.27)) (justify left))
+    )
+    (property "Footprint" "" (at 167.132 150.495 90)
+      (effects (font (size 1.27 1.27)) hide)
+    )
+    (property "Datasheet" "~" (at 168.91 150.495 0)
+      (effects (font (size 1.27 1.27)) hide)
+    )
+    (pin "1")
+    (pin "2")
+    (instances
+      (project "vco"
+        (path "/6034af30-8876-4e85-84ef-45b5f1065c0a"
+          (reference "R5") (unit 1)
+        )
+      )
+    )
+  )
   (symbol (lib_id "Device:R") (at 177.8 113.03 90) (unit 1)
     (in_bom yes) (on_board yes) (dnp no) (fields_autoplaced)
@@
         )
       )
+    )
+  )
+  (symbol (lib_id "Device:R_Potentiometer") (at 252.73 145.415 0) (unit 1)
+    (in_bom yes) (on_board yes) (dnp no) (fields_autoplaced)
+    (property "Reference" "RV1" (at 250.19 144.145 0)
+      (effects (font (size 1.27 1.27)) (justify right))
+    )
+    (property "Value" "R_Potentiometer" (at 250.19 146.685 0)
+      (effects (font (size 1.27 1.27)) (justify right))
+    )
+    (property "Footprint" "" (at 252.73 145.415 0)
+      (effects (font (size 1.27 1.27)) hide)
+    )
+    (property "Datasheet" "~" (at 252.73 145.415 0)
+      (effects (font (size 1.27 1.27)) hide)
+    )
+    (pin "1")
+    (pin "2")
+    (pin "3")
+    (instances
+      (project "vco"
+        (path "/6034af30-8876-4e85-84ef-45b5f1065c0a"
+          (reference "RV1") (unit 1)
+        )
+      )
